File: brd/display/display.sch (KiCad schematic (older format))
At the start: 71 parts, among them P1 CONN_01X09, Q1 2N7002, Q2 2N7002, Q3 2N7002, Q4 2N7002, Q5 2N7002, Q6 2N7002, Q7 2N7002, SW1 SW_PUSH, SW2 SW_PUSH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

Commit message: chg: dev: backup !wip
Parts:
- added D17, D18, D19, D2, D20, D21, D22, D23, D24: RED, LEDs:LED-0805, symbol LED
- added Q8, Q9: 2N7002, Transistors_SMD:sot23, symbol BSS138
- added R31, R33: 100R, Resistors_SMD:R_0805_HandSoldering, symbol R
- added R32, R34: 100k, Resistors_SMD:R_0805_HandSoldering, symbol R
- added R?: 10k, symbol R
Connections:
- net DS_SS: now also R?.1
- net GND: now also Q8.2 (S), Q9.2 (S), R32.1, R34.1, R?.2
- net da: now also D18.1 (A), D2.1 (A); no longer D11.1 (A)
- net db: now also D11.1 (A), D19.1 (A); no longer D12.1 (A)
- net dc: now also D12.1 (A), D20.1 (A); no longer D13.1 (A)
- net dd: now also D17.1 (A), D21.1 (A); no longer D14.1 (A)
- net ddp: now also D16.1 (A)
- net de: now also D13.1 (A), D22.1 (A); no longer D15.1 (A)
- net df: now also D14.1 (A), D23.1 (A); no longer D16.1 (A)
- net dg: now also D15.1 (A), D24.1 (A)
- net dk6: now also D17.2 (K), D2.2 (K)
- net at U2.6 (QG): now also R31.2
- net at U2.7 (QH): now also R33.2
- new net: Q8.1 (G), R31.1, R32.2
- new net: Q9.1 (G), R33.1, R34.2
- new net dk7: D18.2 (K), D19.2 (K), D20.2 (K), D21.2 (K), D22.2 (K), D23.2 (K), D24.2 (K), Q8.3 (D)
- new net dk8: Q9.3 (D)
Other:
- moved on the sheet: C1, C3, C4, C5, C6, C7, C8, C9, D1, D10, D11, D12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
